File: hardware/SharpLCDUSB.kicad_pcb (KiCad board)
At the start: 2 copper layers, 52 x 45 mm, 27 parts, among them J1 A97800TR-ND, J2 Conn_01x10, J3 Conn_01x10, J4 Conn_01x10, J5 Conn_02x05_Odd_Even, SW1 SW_Push, SW2 SW_Push, U1 USBLC6-2SC6, U2 TPS79333-EP, U3 STM32F303CCTx

Commit message: Updated and routed.
Parts:
- added D2: LED, LED_SMD:LED_0603_1608Metric_Pad1.05x0.95mm_HandSolder, F.Cu at (173.2, 81.7)
- added JP1: SolderJumper_2_Bridged, Jumper:SolderJumper-2_P1.3mm_Open_TrianglePad1.0x1.5mm, B.Cu at (142.7, 109.2)
- added JP2: SolderJumper_2_Bridged, Jumper:SolderJumper-2_P1.3mm_Open_TrianglePad1.0x1.5mm, B.Cu at (138.3, 109.2)
- added R2: 330, Resistor_SMD:R_0603_1608Metric_Pad0.98x0.95mm_HandSolder, F.Cu at (173.2, 85.9)
- C1: value 0.1u -> 10u
- J1: footprint digikey-footprints:USB_Micro_B_Female_10103594-0001LF -> KicadFootprint:TE_1981568-1
- moved D1 7.12 mm to (168.4, 81.7), turned to 270 degrees
- moved R1 1.22 mm to (168.4, 85.9), turned to 90 degrees
- moved J5 1.00 mm to (141.0, 83.0)
Connections:
- net /LED renamed /LED1
- U3 pad 20: (no net) -> /LED2
- U3 pad 44: GND -> /BOOT0
Routing:
- net /LED2: track 0.00 -> 26.7 mm, vias 0 -> 2
- net /BOOT0: track 0.00 -> 18.9 mm, vias 0 -> 1
- net VCC: track 92.2 -> 103.8 mm, vias 2 -> 3
- net /SPI_SCK: track 58.8 -> 66.2 mm
- net /SD_CS: track 39.1 -> 45.3 mm
- net /LCD_PWR: track 69.3 -> 75.1 mm
- net /SWDCLK: track 38.4 -> 33.3 mm
- net /NRST: track 68.0 -> 70.7 mm, vias 4 -> 2
- net Net-(D2-Pad2): track 0.00 -> 2.40 mm
- net /LED1: track 25.6 -> 24.3 mm
- net /SWDIO: track 34.6 -> 35.1 mm
- net /LCD_CS: vias 3 -> 4
Other:
- board size 52 x 45 mm -> 52 x 43.6 mm
- board text added: "BTN1"
- board text added: "EXTCOMIN"
- board text added: "GND"
- board text added: "LCD_CS"
- board text added: "LCD_DISP"
- board text added: "LCD_PWR"
- board text added: "RESET"
- board text added: "RX"
- board text added: "SD_CS"
- board text added: "SD_DET"
- board text added: "SPI_MISO"
- board text added: "SPI_MOSI"
- board text added: "SPI_SCK"
- board text added: "SWDIO"
- board text added: "Sharp LCD USB Board Copyright 2021 Nick Butts"
- board text added: "TX"
- board text added: "VCC"
