File: hardware/SharpLCDUSB.sch (KiCad schematic (older format))
At the start: 27 parts, among them J1 A97800TR-ND, J2 Conn_01x10, J3 Conn_01x10, J4 Conn_01x10, J5 Conn_02x05_Odd_Even, SW1 SW_Push, SW2 SW_Push, U1 USBLC6-2SC6, U2 TPS79333-EP, U3 STM32F303CCTx

Commit message: Updated and routed.
Parts:
- added D2: LED, LED_SMD:LED_0603_1608Metric_Pad1.05x0.95mm_HandSolder, symbol Device:LED
- added JP1, JP2: SolderJumper_2_Bridged, Jumper:SolderJumper-2_P1.3mm_Open_TrianglePad1.0x1.5mm, symbol Jumper:SolderJumper_2_Bridged
- added R2: 330, Resistor_SMD:R_0603_1608Metric_Pad0.98x0.95mm_HandSolder, symbol Device:R
- C1: value 0.1u -> 10u
- J1: footprint digikey-footprints:USB_Micro_B_Female_10103594-0001LF -> KicadFootprint:TE_1981568-1
Connections:
- net GND: now also D2.1 (K), JP2.2 (B); no longer U3.44 (BOOT0)
- net VCC: now also JP1.1 (A)
- net LED2: now reaches U3.20 (PB2)
- net LED2: now also R2.1
- net LED renamed LED1
- new net: D2.2 (A), R2.2
- new net BOOT0: JP1.2 (B), JP2.1 (A), U3.44 (BOOT0)
- no-connect marks 25 -> 24
Other:
- moved on the sheet: D1, R1
Changed lines of the file:
@@
 F 0 "J1" H 1514 3223 50  0000 C CNN
 F 1 "A97800TR-ND" H 1514 3132 50  0000 C CNN
-F 2 "digikey-footprints:USB_Micro_B_Female_10103594-0001LF" H 1700 2700 60  0001 L CNN
+F 2 "KicadFootprint:TE_1981568-1" H 1700 2700 60  0001 L CNN
 F 3 "https://cdn.amphenol-icc.com/media/wysiwyg/files/drawing/10103594.pdf" H 1700 2800 60  0001 L CNN
 F 4 "609-4050-1-ND" H 1700 2900 60  0001 L CNN "Digi-Key_PN"
@@
 P 1050 4700
 F 0 "C1" H 1165 4746 50  0000 L CNN
-F 1 "0.1u" H 1165 4655 50  0000 L CNN
+F 1 "10u" H 1165 4655 50  0000 L CNN
 F 2 "Capacitor_SMD:C_0603_1608Metric_Pad1.05x0.95mm_HandSolder" H 1088 4550 50  0001 C CNN
 F 3 "~" H 1050 4700 50  0001 C CNN
@@
 	1    0    0    -1
 $EndComp
-Wire Wire Line
-	6350 2350 5850 2350
-Wire Wire Line
-	5850 2350 5850 2450
 $Comp
 L Device:C C8
@@
 $EndComp
 Wire Wire Line
-	5850 2150 5850 2350
-Connection ~ 5850 2350
-Wire Wire Line
 	6350 2150 6200 2150
 Wire Wire Line
@@
 	6350 4350 5850 4350
 Text Label 5850 4350 0    50   ~ 0
-LED
+LED1
 $Comp
 L Device:LED D1
 U 1 1 6052A84C
-P 4250 6750
-F 0 "D1" V 4289 6632 50  0000 R CNN
-F 1 "LED" V 4198 6632 50  0000 R CNN
-F 2 "LED_SMD:LED_0603_1608Metric_Pad1.05x0.95mm_HandSolder" H 4250 6750 50  0001 C CNN
-F 3 "~" H 4250 6750 50  0001 C CNN
-F 4 "475-2709-1-ND" H 4250 6750 50  0001 C CNN "Digi-Key_PN"
-	1    4250 6750
+P 3650 6750
+F 0 "D1" V 3689 6632 50  0000 R CNN
+F 1 "LED" V 3598 6632 50  0000 R CNN
+F 2 "LED_SMD:LED_0603_1608Metric_Pad1.05x0.95mm_HandSolder" H 3650 6750 50  0001 C CNN
+F 3 "~" H 3650 6750 50  0001 C CNN
+F 4 "475-2709-1-ND" H 3650 6750 50  0001 C CNN "Digi-Key_PN"
+	1    3650 6750
 	0    -1   -1   0
 $EndComp
@@
 L Device:R R1
 U 1 1 6052B05C
-P 4250 6300
-F 0 "R1" H 4320 6346 50  0000 L CNN
-F 1 "330" H 4320 6255 50  0000 L CNN
-F 2 "Resistor_SMD:R_0603_1608Metric_Pad0.98x0.95mm_HandSolder" V 4180 6300 50  0001 C CNN
-F 3 "~" H 4250 6300 50  0001 C CNN
-	1    4250 6300
+P 3650 6300
+F 0 "R1" H 3720 6346 50  0000 L CNN
+F 1 "330" H 3720 6255 50  0000 L CNN
+F 2 "Resistor_SMD:R_0603_1608Metric_Pad0.98x0.95mm_HandSolder" V 3580 6300 50  0001 C CNN
+F 3 "~" H 3650 6300 50  0001 C CNN
+	1    3650 6300
 	1    0    0    -1
 $EndComp
@@
 L power:GND #PWR014
 U 1 1 6052B8CC
-P 4250 7050
-F 0 "#PWR014" H 4250 6800 50  0001 C CNN
-F 1 "GND" H 4255 6877 50  0000 C CNN
-F 2 "" H 4250 7050 50  0001 C CNN
-F 3 "" H 4250 7050 50  0001 C CNN
-	1    4250 7050
-	1    0    0    -1
-$EndComp
-Wire Wire Line
-	4250 6900 4250 7050
-Wire Wire Line
-	4250 6600 4250 6450
-Wire Wire Line
-	4250 6150 4250 6050
-Wire Wire Line
-	4250 6050 4000 6050
-Text Label 4000 6050 0    50   ~ 0
-LED
+P 3650 7050
+F 0 "#PWR014" H 3650 6800 50  0001 C CNN
+F 1 "GND" H 3655 6877 50  0000 C CNN
+F 2 "" H 3650 7050 50  0001 C CNN
+F 3 "" H 3650 7050 50  0001 C CNN
+	1    3650 7050
+	1    0    0    -1
+$EndComp
+Wire Wire Line
+	3650 6900 3650 7050
+Wire Wire Line
+	3650 6600 3650 6450
+Wire Wire Line
+	3650 6150 3650 6050
+Wire Wire Line
+	3650 6050 3400 6050
+Text Label 3400 6050 0    50   ~ 0
+LED1
 NoConn ~ 6350 2550
 NoConn ~ 6350 2650
@@
 NoConn ~ 6350 3050
 NoConn ~ 6350 3350
-NoConn ~ 6350 3450
 NoConn ~ 6350 3550
 NoConn ~ 6350 3650
@@
 	6350 2850 5250 2850
 Connection ~ 5250 2850
+$Comp
+L Jumper:SolderJumper_2_Bridged JP2
+U 1 1 604A9A42
+P 2050 6950
+F 0 "JP2" V 2004 7018 50  0000 L CNN
+F 1 "SolderJumper_2_Bridged" V 2095 7018 50  0000 L CNN
+F 2 "Jumper:SolderJumper-2_P1.3mm_Open_TrianglePad1.0x1.5mm" H 2050 6950 50  0001 C CNN
+F 3 "~" H 2050 6950 50  0001 C CNN
+	1    2050 6950
+	0    1    1    0
+$EndComp
+Wire Wire Line
+	5850 2150 5850 2450
+Wire Wire Line
+	6350 2350 6000 2350
+Text Label 6000 2350 0    50   ~ 0
+BOOT0
+$Comp
+L power:GND #PWR020
+U 1 1 604B548E
+P 2050 7250
+F 0 "#PWR020" H 2050 7000 50  0001 C CNN
+F 1 "GND" H 2055 7077 50  0000 C CNN
+F 2 "" H 2050 7250 50  0001 C CNN
+F 3 "" H 2050 7250 50  0001 C CNN
+	1    2050 7250
+	1    0    0    -1
+$EndComp
+$Comp
+L Jumper:SolderJumper_2_Bridged JP1
+U 1 1 604B62CD
+P 2050 6300
+F 0 "JP1" V 2004 6368 50  0000 L CNN
+F 1 "SolderJumper_2_Bridged" V 2095 6368 50  0000 L CNN
+F 2 "Jumper:SolderJumper-2_P1.3mm_Open_TrianglePad1.0x1.5mm" H 2050 6300 50  0001 C CNN
+F 3 "~" H 2050 6300 50  0001 C CNN
+	1    2050 6300
+	0    1    1    0
+$EndComp
+$Comp
+L power:VCC #PWR019
+U 1 1 604B6A47
+P 2050 6000
+F 0 "#PWR019" H 2050 5850 50  0001 C CNN
+F 1 "VCC" H 2065 6173 50  0000 C CNN
+F 2 "" H 2050 6000 50  0001 C CNN
+F 3 "" H 2050 6000 50  0001 C CNN
+	1    2050 6000
+	1    0    0    -1
+$EndComp
+Wire Wire Line
+	2050 6000 2050 6150
+Wire Wire Line
+	2050 7100 2050 7250
+Wire Wire Line
+	2050 6800 2050 6650
+Wire Wire Line
+	2050 6650 1550 6650
+Connection ~ 2050 6650
+Wire Wire Line
+	2050 6650 2050 6450
+Text Label 1550 6650 0    50   ~ 0
+BOOT0
+$Comp
+L Device:LED D2
+U 1 1 604F6C01
+P 4400 6750
+F 0 "D2" V 4439 6632 50  0000 R CNN
+F 1 "LED" V 4348 6632 50  0000 R CNN
+F 2 "LED_SMD:LED_0603_1608Metric_Pad1.05x0.95mm_HandSolder" H 4400 6750 50  0001 C CNN
+F 3 "~" H 4400 6750 50  0001 C CNN
+F 4 "475-2709-1-ND" H 4400 6750 50  0001 C CNN "Digi-Key_PN"
+	1    4400 6750
+	0    -1   -1   0
+$EndComp
+$Comp
+L Device:R R2
+U 1 1 604F7069
+P 4400 6300
+F 0 "R2" H 4470 6346 50  0000 L CNN
+F 1 "330" H 4470 6255 50  0000 L CNN
+F 2 "Resistor_SMD:R_0603_1608Metric_Pad0.98x0.95mm_HandSolder" V 4330 6300 50  0001 C CNN
+F 3 "~" H 4400 6300 50  0001 C CNN
+	1    4400 6300
+	1    0    0    -1
+$EndComp
+$Comp
+L power:GND #PWR0102
+U 1 1 604F7073
+P 4400 7050
+F 0 "#PWR0102" H 4400 6800 50  0001 C CNN
+F 1 "GND" H 4405 6877 50  0000 C CNN
+F 2 "" H 4400 7050 50  0001 C CNN
+F 3 "" H 4400 7050 50  0001 C CNN
+	1    4400 7050
+	1    0    0    -1
+$EndComp
+Wire Wire Line
+	4400 6900 4400 7050
+Wire Wire Line
+	4400 6600 4400 6450
+Wire Wire Line
+	4400 6150 4400 6050
+Wire Wire Line
+	4400 6050 4150 6050
+Text Label 4150 6050 0    50   ~ 0
+LED2
+Wire Wire Line
+	6350 3450 5900 3450
+Text Label 5900 3450 0    50   ~ 0
+LED2
 $EndSCHEMATC
